Commit message: 1

File: src/ur5_t2_4230/models/urdf/blue_box.urdf (robot description, URDF)
Before this commit: robot blue_box, 1 links, 0 joints
Links:
- link base_link: geometry collision box size=0.05 0.05 0.05; visual box size=0.05 0.05 0.05

File: src/ur5_t2_4230/models/urdf/blue_cylinder.urdf (robot description, URDF)
Before this commit: robot blue_cylinder, 1 links, 0 joints
Links:
- link base_link: geometry collision cylinder length=0.1 radius=0.025; visual cylinder length=0.05 radius=0.025

File: src/ur5_t2_4230/models/urdf/green_box.urdf (robot description, URDF)
Before this commit: robot green_box, 1 links, 0 joints
Links:
- link base_link: geometry collision box size=0.05 0.05 0.05; visual box size=0.05 0.05 0.05

File: src/ur5_t2_4230/models/urdf/green_cylinder.urdf (robot description, URDF)
Before this commit: robot green_cylinder, 1 links, 0 joints
Links:
- link base_link: geometry collision cylinder length=0.05 radius=0.025; visual cylinder length=0.05 radius=0.025

File: src/ur5_t2_4230/models/urdf/red_box.urdf (robot description, URDF)
Before this commit: robot red_box, 1 links, 0 joints
Links:
- link base_link: geometry collision box size=0.05 0.05 0.05; visual box size=0.05 0.05 0.05

File: src/ur5_t2_4230/models/urdf/red_cylinder.urdf (robot description, URDF)
Before this commit: robot red_cylinder, 1 links, 0 joints
Links:
- link base_link: geometry collision cylinder length=0.05 radius=0.025; visual cylinder length=0.05 radius=0.025
